File: board/wakeup.brd (EAGLE design)
At the start: 65 x 56 mm, 24 parts, among them IC2 ATMEGA48/88/168-AU, K1 PIN20X2, U1 EEPROM24

Commit message: Fixed some naming and added tag
Parts:
- renumbered U$1 to UR4, U$2 to UR3, U$3 to UR6, U$4 to UR5, U$5 to UR7, U$6 to UR8, U$7 to UR2, U$8 to UR1
Other:
- board text added: "2018 RB MS"
Changed lines of the file:
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@@
 <wire x1="46" y1="4" x2="45" y2="3" width="0" layer="20" curve="-90"/>
 <wire x1="44" y1="4" x2="45" y2="3" width="0" layer="20" curve="90"/>
+<text x="18" y="1" size="1.9304" layer="1" font="vector">2018 RB MS</text>
 </plain>
 <attributes>
@@
 <attribute name="VALUE" x="40.54" y="30.73" size="1.27" layer="27" rot="R90"/>
 </element>
-<element name="U$7" library="1" package="SOT" value="AMC7135" x="32" y="31" smashed="yes" rot="R270">
+<element name="UR2" library="1" package="SOT" value="AMC7135" x="32" y="31" smashed="yes" rot="R270">
 <attribute name="NAME" x="30.46" y="32.405" size="1.27" layer="25"/>
 <attribute name="VALUE" x="26.3851" y="33.4051" size="1.27" layer="27" rot="R270"/>
 </element>
-<element name="U$8" library="1" package="SOT" value="AMC7135" x="23" y="31" smashed="yes" rot="R270">
+<element name="UR1" library="1" package="SOT" value="AMC7135" x="23" y="31" smashed="yes" rot="R270">
 <attribute name="NAME" x="21.46" y="27.905" size="1.27" layer="25"/>
 <attribute name="VALUE" x="17.3851" y="33.4051" size="1.27" layer="27" rot="R270"/>
 </element>
-<element name="U$1" library="1" package="SOT" value="AMC7135" x="32" y="26" smashed="yes" rot="R270">
+<element name="UR4" library="1" package="SOT" value="AMC7135" x="32" y="26" smashed="yes" rot="R270">
 <attribute name="NAME" x="30.46" y="27.405" size="1.27" layer="25"/>
 <attribute name="VALUE" x="26.3851" y="28.4051" size="1.27" layer="27" rot="R270"/>
 </element>
-<element name="U$2" library="1" package="SOT" value="AMC7135" x="23" y="26" smashed="yes" rot="R270">
+<element name="UR3" library="1" package="SOT" value="AMC7135" x="23" y="26" smashed="yes" rot="R270">
 <attribute name="NAME" x="21.46" y="22.905" size="1.27" layer="25"/>
 <attribute name="VALUE" x="17.3851" y="28.4051" size="1.27" layer="27" rot="R270"/>
 </element>
-<element name="U$3" library="1" package="SOT" value="AMC7135" x="32" y="21" smashed="yes" rot="R270">
+<element name="UR6" library="1" package="SOT" value="AMC7135" x="32" y="21" smashed="yes" rot="R270">
 <attribute name="NAME" x="30.46" y="22.405" size="1.27" layer="25"/>
 <attribute name="VALUE" x="26.3851" y="23.4051" size="1.27" layer="27" rot="R270"/>
 </element>
-<element name="U$4" library="1" package="SOT" value="AMC7135" x="23" y="21" smashed="yes" rot="R270">
+<element name="UR5" library="1" package="SOT" value="AMC7135" x="23" y="21" smashed="yes" rot="R270">
 <attribute name="NAME" x="21.46" y="17.905" size="1.27" layer="25"/>
 <attribute name="VALUE" x="17.3851" y="23.4051" size="1.27" layer="27" rot="R270"/>
 </element>
-<element name="U$5" library="1" package="SOT" value="AMC7135" x="23" y="16" smashed="yes" rot="R270">
+<element name="UR7" library="1" package="SOT" value="AMC7135" x="23" y="16" smashed="yes" rot="R270">
 <attribute name="NAME" x="21.46" y="12.905" size="1.27" layer="25"/>
 <attribute name="VALUE" x="17.3851" y="18.4051" size="1.27" layer="27" rot="R270"/>
 </element>
-<element name="U$6" library="1" package="SOT" value="AMC7135" x="32" y="16" smashed="yes" rot="R270">
+<element name="UR8" library="1" package="SOT" value="AMC7135" x="32" y="16" smashed="yes" rot="R270">
 <attribute name="NAME" x="30.46" y="17.405" size="1.27" layer="25"/>
 <attribute name="VALUE" x="26.3851" y="18.4051" size="1.27" layer="27" rot="R270"/>
@@
 <contactref element="SL2" pad="2"/>
 <contactref element="SV1" pad="6"/>
-<contactref element="U$7" pad="2"/>
-<contactref element="U$7" pad="2@1"/>
-<contactref element="U$8" pad="2"/>
-<contactref element="U$8" pad="2@1"/>
-<contactref element="U$1" pad="2"/>
-<contactref element="U$1" pad="2@1"/>
-<contactref element="U$2" pad="2"/>
-<contactref element="U$2" pad="2@1"/>
-<contactref element="U$3" pad="2"/>
-<contactref element="U$3" pad="2@1"/>
-<contactref element="U$4" pad="2"/>
-<contactref element="U$4" pad="2@1"/>
-<contactref element="U$5" pad="2"/>
-<contactref element="U$5" pad="2@1"/>
-<contactref element="U$6" pad="2"/>
-<contactref element="U$6" pad="2@1"/>
+<contactref element="UR2" pad="2"/>
+<contactref element="UR2" pad="2@1"/>
+<contactref element="UR1" pad="2"/>
+<contactref element="UR1" pad="2@1"/>
+<contactref element="UR4" pad="2"/>
+<contactref element="UR4" pad="2@1"/>
+<contactref element="UR3" pad="2"/>
+<contactref element="UR3" pad="2@1"/>
+<contactref element="UR6" pad="2"/>
+<contactref element="UR6" pad="2@1"/>
+<contactref element="UR7" pad="2"/>
+<contactref element="UR7" pad="2@1"/>
+<contactref element="UR8" pad="2"/>
+<contactref element="UR8" pad="2@1"/>
 <contactref element="C3" pad="2"/>
 <wire x1="62.075" y1="32.4975" x2="61.865" y2="32.7075" width="0.4064" layer="1"/>
@@
 <via x="35" y="31" extent="1-16" drill="0.9" shape="square"/>
 <via x="35" y="26" extent="1-16" drill="0.9" shape="square"/>
-<via x="35" y="21" extent="1-16" drill="0.9" shape="square"/>
 <via x="35" y="16" extent="1-16" drill="0.9" shape="square"/>
 <wire x1="35" y1="16" x2="31.67" y2="16" width="0.6096" layer="1"/>
-<wire x1="22.67" y1="21" x2="35" y2="21" width="0.6096" layer="1"/>
 <contactref element="CREE_LED1" pad="HT"/>
 <wire x1="28.4083875" y1="43.246209375" x2="24.246209375" y2="43.246209375" width="0.4064" layer="1"/>
@@
 <wire x1="22.67" y1="31" x2="35" y2="31" width="0.6096" layer="1"/>
 <wire x1="22" y1="26" x2="35" y2="26" width="0.6096" layer="1"/>
+<contactref element="UR5" pad="2"/>
+<contactref element="UR5" pad="2@1"/>
+<via x="35" y="21" extent="1-16" drill="0.9" shape="square"/>
+<wire x1="22.67" y1="21" x2="35" y2="21" width="0.6096" layer="1"/>
+<wire x1="61.865" y1="36.625" x2="61.865" y2="37.895" width="0" layer="19" extent="1-1"/>
+<wire x1="61.865" y1="35.355" x2="61.865" y2="36.625" width="0" layer="19" extent="1-1"/>
+<wire x1="61.865" y1="39.165" x2="61.865" y2="37.895" width="0" layer="19" extent="1-1"/>
+<wire x1="38" y1="35" x2="38" y2="35.05" width="0" layer="19" extent="1-1"/>
+<wire x1="22.67" y1="26" x2="22" y2="26" width="0" layer="19" extent="1-1"/>
+<wire x1="24" y1="41" x2="24.260740625" y2="40.260740625" width="0" layer="19" extent="1-1"/>
+<wire x1="20.003" y1="26" x2="22" y2="26" width="0" layer="19" extent="1-1"/>
+<wire x1="20.003" y1="31" x2="22.67" y2="31" width="0" layer="19" extent="1-1"/>
+<wire x1="20.003" y1="21" x2="22.67" y2="21" width="0" layer="19" extent="1-1"/>
+<wire x1="29.003" y1="16" x2="31.67" y2="16" width="0" layer="19" extent="1-1"/>
+<wire x1="22.67" y1="16" x2="22" y2="16" width="0" layer="19" extent="1-1"/>
+<wire x1="20.003" y1="16" x2="22" y2="16" width="0" layer="19" extent="1-1"/>
+<wire x1="32" y1="31.33" x2="35" y2="31" width="0" layer="19" extent="1-1"/>
+<wire x1="29.003" y1="31" x2="31.67" y2="31" width="0" layer="19" extent="1-1"/>
+<wire x1="31.67" y1="26" x2="35" y2="26" width="0" layer="19" extent="1-1"/>
+<wire x1="29.003" y1="26" x2="31.67" y2="26" width="0" layer="19" extent="1-1"/>
+<wire x1="31.67" y1="21" x2="35" y2="21" width="0" layer="19" extent="1-1"/>
+<wire x1="29.003" y1="21" x2="31.67" y2="21" width="0" layer="19" extent="1-1"/>
 </signal>
 <signal name="+3V3">
@@
 </signal>
 <signal name="RED_LED">
-<contactref element="U$8" pad="3"/>
-<contactref element="U$7" pad="3"/>
+<contactref element="UR1" pad="3"/>
+<contactref element="UR2" pad="3"/>
 <contactref element="IC2" pad="9"/>
 <wire x1="19.749" y1="29.501" x2="28.749" y2="29.501" width="0.6096" layer="1"/>
@@
 </signal>
 <signal name="GREEN_LED">
-<contactref element="U$2" pad="3"/>
-<contactref element="U$1" pad="3"/>
+<contactref element="UR3" pad="3"/>
+<contactref element="UR4" pad="3"/>
 <contactref element="IC2" pad="10"/>
 <wire x1="19.749" y1="24.501" x2="28.749" y2="24.501" width="0.6096" layer="1"/>
@@
 </signal>
 <signal name="BLUE_LED">
-<contactref element="U$4" pad="3"/>
-<contactref element="U$3" pad="3"/>
 <contactref element="IC2" pad="13"/>
+<wire x1="45.4" y1="26.15665" x2="45.4" y2="27.7074" width="0.4064" layer="1"/>
+<contactref element="UR5" pad="3"/>
+<contactref element="UR6" pad="3"/>
 <wire x1="19.749" y1="19.501" x2="28.749" y2="19.501" width="0.6096" layer="1"/>
 <wire x1="28.749" y1="19.501" x2="38.74435" y2="19.501" width="0.4064" layer="1"/>
 <wire x1="38.74435" y1="19.501" x2="45.4" y2="26.15665" width="0.4064" layer="1"/>
-<wire x1="45.4" y1="26.15665" x2="45.4" y2="27.7074" width="0.4064" layer="1"/>
 </signal>
 <signal name="WHITE_LED">
-<contactref element="U$6" pad="3"/>
-<contactref element="U$5" pad="3"/>
+<contactref element="UR8" pad="3"/>
+<contactref element="UR7" pad="3"/>
 <contactref element="IC2" pad="14"/>
 <wire x1="19.749" y1="14.501" x2="28.749" y2="14.501" width="0.6096" layer="1"/>
@@
 </signal>
 <signal name="GREEN_LED_OUT">
-<contactref element="U$1" pad="1"/>
-<contactref element="U$2" pad="1"/>
+<contactref element="UR4" pad="1"/>
+<contactref element="UR3" pad="1"/>
 <wire x1="28.749" y1="27.499" x2="19.749" y2="27.499" width="0.6096" layer="1"/>
 <contactref element="SL1" pad="7"/>
@@
 </signal>
 <signal name="BLUE_LED_OUT">
-<contactref element="U$3" pad="1"/>
-<contactref element="U$4" pad="1"/>
+<contactref element="UR6" pad="1"/>
+<contactref element="UR5" pad="1"/>
 <wire x1="28.749" y1="22.499" x2="19.749" y2="22.499" width="0.6096" layer="1"/>
 <contactref element="SL1" pad="6"/>
@@
 </signal>
 <signal name="WHITE_LED_OUT">
-<contactref element="U$5" pad="1"/>
-<contactref element="U$6" pad="1"/>
+<contactref element="UR7" pad="1"/>
+<contactref element="UR8" pad="1"/>
 <wire x1="28.749" y1="17.499" x2="19.749" y2="17.499" width="0.6096" layer="1"/>
 <contactref element="SL1" pad="5"/>
@@
 </signal>
 <signal name="RED_LED_OUT">
-<contactref element="U$7" pad="1"/>
-<contactref element="U$8" pad="1"/>
+<contactref element="UR2" pad="1"/>
+<contactref element="UR1" pad="1"/>
 <wire x1="19.749" y1="32.499" x2="28.749" y2="32.499" width="0.6096" layer="1"/>
 <contactref element="SL1" pad="8"/>

Commit message: Much better
Parts:
- removed C2: 47nF, rcl:C0805
- removed CREE_LED1: CREE_XL_MCE, CreeXL-MC-E:CREE_XL_MCE
- removed J1: (no value), con-jack:SPC4078
- removed UR1, UR2, UR3, UR4, UR5, UR6, UR7, UR8: AMC7135, 1:SOT
- added C4: 100nF, rcl:C0603
- added C5, C6, C7: 10µF, rcl:C0805
- added CREE_LED2: CREE_XL_MCE, CreeXL-MC-E:CREE_XL_MCE
- added Q5, Q6, Q7, Q8: BC846BSMD, transistor-npn:SOT23
- added R12, R13, R14, R15: 1k, resistor:R0603
- added R18, R19, R4, R5: 1k, resistor:M0805
- added SL4, SL5, SL6: (no value), con-amp-quick:04P
- added UR10, UR11, UR12, UR13, UR14, UR15, UR16, UR9: AMC7135, 1:SOT
- C3: value 47nF -> 100nF; device rcl:C0805 -> rcl:C0603
- SL2: device con-amp-quick:02P -> con-amp-quick:04P
- moved SL2 34.5 mm to (52.5, 8.80), turned to 180 degrees
- moved C3 3.32 mm to (38.9, 32.8), turned to 90 degrees
Connections:
- new net ADC0: IC2.23, SL5.2
- new net GLUMP1: Q5.3, R15.1, UR10.3, UR9.3
- new net N$4: C4.1, IC2.20
- new net N$5: Q8.1, R19.1
- new net N$6: Q7.1, R18.1
- new net N$7: Q5.1, R5.1
- new net N$8: Q6.1, R4.1
- new net SCHMARN1: Q6.3, R14.1, UR11.3, UR12.3
- new net TEST1: Q7.3, R12.1, UR13.3, UR14.3
- new net WHITE_LED1: R19.2
- new net ZEUCH1: Q8.3, R13.1, UR15.3, UR16.3
- net +3V3: now also IC2.18, SL5.3; no longer C2.1, SL2.1
- net +5V: now also C5.1, C6.1, C7.1, CREE_LED2.1, CREE_LED2.2, CREE_LED2.3, CREE_LED2.4, CREE_LED2.HT, R12.2, R13.2, R14.2, R15.2, SL4.3, SL4.4, SL5.4; no longer J1.3
- net BLUE_LED: now also R18.2; no longer UR5.3, UR6.3
- net BLUE_LED_OUT: now also CREE_LED2.7, UR13.1, UR14.1; no longer CREE_LED1.3, UR5.1, UR6.1
- net GND: now also C4.2, C5.2, C6.2, C7.2, Q5.2, Q6.2, Q7.2, Q8.2, SL4.1, SL4.2, SL5.1, UR10.2, UR10.2@1, UR11.2, UR11.2@1, UR12.2, UR12.2@1, UR13.2, UR13.2@1, UR14.2, UR14.2@1, UR15.2, UR15.2@1, UR16.2, UR16.2@1, UR9.2, UR9.2@1; no longer C2.2, CREE_LED1.5, CREE_LED1.6, CREE_LED1.7, CREE_LED1.8, CREE_LED1.HT, J1.1, J1.2, SL2.2, UR1.2, UR1.2@1, UR2.2, UR2.2@1, UR3.2, UR3.2@1, UR4.2, UR4.2@1, UR5.2, UR5.2@1, UR6.2, UR6.2@1, UR7.2, UR7.2@1, UR8.2, UR8.2@1
- net GREEN_LED: now also R4.2; no longer UR3.3, UR4.3
- net GREEN_LED_OUT: now also CREE_LED2.6, UR11.1, UR12.1; no longer CREE_LED1.2, UR3.1, UR4.1
- net I2C_SCL1: now also IC2.28; no longer IC2.24
- net I2C_SDA1: now also IC2.27; no longer IC2.23
- net RED_LED: now also R5.2; no longer UR1.3, UR2.3
- net RED_LED_OUT: now also CREE_LED2.5, UR10.1, UR9.1; no longer CREE_LED1.1, UR1.1, UR2.1
- net WHITE_LED: no longer UR7.3, UR8.3
- net WHITE_LED_OUT: now also CREE_LED2.8, UR15.1, UR16.1; no longer CREE_LED1.4, UR7.1, UR8.1
Routing:
- net +5V: track 73.5 -> 223.9 mm
- net +3V3: track 148.2 -> 208.8 mm
- net WHITE_LED: track 34.0 -> 8.04 mm
- net I2C_SCL1: track 71.7 -> 45.8 mm
- net RED_LED: track 25.3 -> 3.12 mm
- net GND: track 100.5 -> 79.9 mm, vias 10 -> 13
- net GLUMP1: track 0.00 -> 20.2 mm
- net GREEN_LED: track 25.5 -> 5.31 mm
- net BLUE_LED: track 30.0 -> 10.5 mm
- net SCHMARN1: track 0.00 -> 18.7 mm
- net TEST1: track 0.00 -> 17.8 mm
- net ZEUCH1: track 0.00 -> 17.2 mm
- net I2C_SDA1: track 62.0 -> 49.8 mm
- net N$3: track 6.53 -> 13.2 mm
- net GREEN_LED_OUT: track 37.8 -> 31.7 mm
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
Commit message: Fixed some errors
Parts:
- moved Q6 0.22 mm to (34.0, 25.1)
- moved R14 0.20 mm to (32.4, 23.5)
- moved Q5 0.14 mm to (34.0, 28.3)
Connections:
- removed net WHITE_LED1: R19.2
- net WHITE_LED: now also R19.2
Routing:
- net +5V: track 223.9 -> 233.4 mm
- net WHITE_LED: track 8.04 -> 12.5 mm
- net GND: track 79.9 -> 75.9 mm, vias 13 -> 15
- net +3V3: track 208.8 -> 206.6 mm
- net SDA0_I2C_ID_EEPROM: track 32.6 -> 31.6 mm
- net WHITE_LED_OUT: track 47.6 -> 46.6 mm
- net GLUMP1: track 20.2 -> 21.1 mm
- net SCHMARN1: track 18.7 -> 18.0 mm
- net TEST1: track 17.8 -> 17.1 mm

Commit message: Finalized Updates
Connections:
- net GLUMP1 renamed RED_POWER
- net SCHMARN1 renamed GREEN_POWER
- net TEST1 renamed BLUE_POWER
- net ZEUCH1 renamed WHITE_POWER
Routing:
- net ADC0: track 0.00 -> 35.2 mm, vias 0 -> 1
- net +5V: track 233.4 -> 231.3 mm
- net WHITE_LED_OUT: track 46.6 -> 47.2 mm
